Commit message: robot model update

File: urdf/robot.xacro (robot description, xacro)
@@ -16,4 +16,5 @@
      	</geometry>
 	</xacro:macro>
+	<!--#################  MATERIAL PROPERTIES  ############## -->
   <material name="black">
     <color rgba="0.0 0.0 0.0 1.0"/>
@@ -40,4 +41,5 @@
     <color rgba="1.0 1.0 1.0 1.0"/>
   </material>
+  <!--#################  LINK PROPERTIES  ############## -->
 	  <link name="link_chassis">
     <!-- pose and inertial -->
@@ -61,5 +63,5 @@
       <material name="blue"/>
     </visual>
-    <!-- caster front -->
+    <!-- caster front
     <collision name="caster_front_collision">
       <origin rpy=" 0 0 0" xyz="0.35 0 -0.05"/>
@@ -73,73 +75,173 @@
         <sphere radius="0.05"/>
       </geometry>
-    </visual>
-  </link>
-   <link name="link_right_wheel">
-    <xacro:default_inertial mass="0.2"/>
-    <collision name="link_right_wheel_collision">
-      <origin rpy="0 1.5707 1.5707" xyz="0 0 0"/>
-      <xacro:wheel_geometry />
-    </collision>
-    <visual name="link_right_wheel_visual">
-      <origin rpy="0 1.5707 1.5707" xyz="0 0 0"/>
-      <xacro:wheel_geometry />
-      <material name="red"/>
-    </visual>
-  </link>
-   <link name="link_left_wheel">
-    <xacro:default_inertial mass="0.2"/>
-    <collision name="link_left_wheel_collision">
-      <origin rpy="0 1.5707 1.5707" xyz="0 0 0"/>
-      <xacro:wheel_geometry />
-    </collision>
-    <visual name="link_left_wheel_visual">
-      <origin rpy="0 1.5707 1.5707" xyz="0 0 0"/>
-      <xacro:wheel_geometry />
-      <material name="red"/>
-    </visual>
-  </link>
-  <joint name="joint_right_wheel" type="continuous">
-    <origin rpy="0 0 0" xyz="-0.05 0.15 0"/>
-    <child link="link_right_wheel"/>
-    <parent link="link_chassis"/>
-    <axis rpy="0 0 0" xyz="0 1 0"/>
-    <limit effort="10000" velocity="1000"/>
-    <joint_properties damping="1.0" friction="1.0"/>
-  </joint>
-  <joint name="joint_left_wheel" type="continuous">
-    <origin rpy="0 0 0" xyz="-0.05 -0.15 0"/>
-    <child link="link_left_wheel"/>
-    <parent link="link_chassis"/>
-    <axis rpy="0 0 0" xyz="0 1 0"/>
-    <limit effort="10000" velocity="1000"/>
-    <joint_properties damping="1.0" friction="1.0"/>
-  </joint>
+    </visual>-->
+  </link>
+  <link name="link_back_right_wheel">
+    <xacro:default_inertial mass="0.2"/>
+    <collision name="link_back_right_wheel_collision">
+      <origin rpy="0 1.5707 1.5707" xyz="0 0 0"/>
+      <xacro:wheel_geometry />
+    </collision>
+    <visual name="link_back_right_wheel_visual">
+      <origin rpy="0 1.5707 1.5707" xyz="0 0 0"/>
+      <xacro:wheel_geometry />
+      <material name="red"/>
+    </visual>
+  </link>
+   <link name="link_back_left_wheel">
+    <xacro:default_inertial mass="0.2"/>
+    <collision name="link_back_left_wheel_collision">
+      <origin rpy="0 1.5707 1.5707" xyz="0 0 0"/>
+      <xacro:wheel_geometry />
+    </collision>
+    <visual name="link_back_left_wheel_visual">
+      <origin rpy="0 1.5707 1.5707" xyz="0 0 0"/>
+      <xacro:wheel_geometry />
+      <material name="red"/>
+    </visual>
+  </link>
+   <link name="link_front_right_wheel">
+    <xacro:default_inertial mass="0.2"/>
+    <collision name="link_front_right_wheel_collision">
+      <origin rpy="0 1.5707 1.5707" xyz="0 0 0"/>
+      <xacro:wheel_geometry />
+    </collision>
+    <visual name="link_front_right_wheel_visual">
+      <origin rpy="0 1.5707 1.5707" xyz="0 0 0"/>
+      <xacro:wheel_geometry />
+      <material name="red"/>
+    </visual>
+  </link>
+   <link name="link_front_left_wheel">
+    <xacro:default_inertial mass="0.2"/>
+    <collision name="link_front_left_wheel_collision">
+      <origin rpy="0 1.5707 1.5707" xyz="0 0 0"/>
+      <xacro:wheel_geometry />
+    </collision>
+    <visual name="link_front_left_wheel_visual">
+      <origin rpy="0 1.5707 1.5707" xyz="0 0 0"/>
+      <xacro:wheel_geometry />
+      <material name="red"/>
+    </visual>
+  </link>
+  <joint name="joint_back_right_wheel" type="continuous">
+    <origin rpy="0 0 0" xyz="-0.20 0.15 0"/>
+    <child link="link_back_right_wheel"/>
+    <parent link="link_chassis"/>
+    <axis rpy="0 0 0" xyz="0 1 0"/>
+    <limit effort="10000" velocity="1000"/>
+    <joint_properties damping="1.0" friction="1.0"/>
+  </joint>
+  <joint name="joint_back_left_wheel" type="continuous">
+    <origin rpy="0 0 0" xyz="-0.20 -0.15 0"/>
+    <child link="link_back_left_wheel"/>
+    <parent link="link_chassis"/>
+    <axis rpy="0 0 0" xyz="0 1 0"/>
+    <limit effort="10000" velocity="1000"/>
+    <joint_properties damping="1.0" friction="1.0"/>
+  </joint>
+  <joint name="joint_front_right_wheel" type="continuous">
+    <origin rpy="0 0 0" xyz="0.20 0.15 0"/>
+    <child link="link_front_right_wheel"/>
+    <parent link="link_chassis"/>
+    <axis rpy="0 0 0" xyz="0 1 0"/>
+    <limit effort="10000" velocity="1000"/>
+    <joint_properties damping="1.0" friction="1.0"/>
+  </joint>
+  <joint name="joint_front_left_wheel" type="continuous">
+    <origin rpy="0 0 0" xyz="0.20 -0.15 0"/>
+    <child link="link_front_left_wheel"/>
+    <parent link="link_chassis"/>
+    <axis rpy="0 0 0" xyz="0 1 0"/>
+    <limit effort="10000" velocity="1000"/>
+    <joint_properties damping="1.0" friction="1.0"/>
+  </joint>
+<!--camera links - neck definition -->
+  <link name="neck_base_link">
+  	<inertial>
+  		<mass value="0.01"/>
+  		<origin xyz="0 0 0" rpy="0 0 0" />
+  		<inertia ixx="0.0000416666667" ixy="0" ixz="0" iyy="0.0000416666667" iyz="0" izz="0.0000416666667"/>
+  	</inertial>
+  	<collision>
+  	  <origin xyz="0 0 0" rpy="0 0 0"/>
+      <geometry>
+        <box size="0.1 0.1 0.1"/>
+      </geometry>
+  	</collision>
+  	<visual>
+  	  <origin xyz="0 0 0" rpy="0 0 0"/>
+      <geometry>
+        <box size="0.1 0.1 0.1"/>
+      </geometry>
+      <material name="red" />
+  	</visual>
+  </link>
+  <joint name="neck_base_to_chassis" type="fixed">
+  	<origin rpy="0 0 0" xyz="0 0 0.085"/>
+  	<parent link="link_chassis"/>
+  	<child link="neck_base_link"/>
+  </joint>
+  <link name="neck_link">
+  	<inertial>
+  		<mass value="0.00125"/>
+  		<origin xyz="0 0 0" rpy="0 0 0" />
+  		<inertia ixx="0.000010279" ixy="0" ixz="0" iyy="0.000010279" iyz="0" izz="0.000007225"/>
+  	</inertial>
+  	<collision>
+  	  <origin xyz="0 0 0.125" rpy="0 0 0"/>
+      <geometry>
+        <cylinder radius="0.04" length="0.25"/>
+      </geometry>
+  	</collision>
+  	<visual>
+  	  <origin xyz="0 0 0.125" rpy="0 0 0"/>
+      <geometry>
+        <cylinder radius="0.04" length="0.25"/>
+      </geometry>
+      <material name="red" />
+  	</visual>
+  </link>
   <link name="camera_link">
-	    <collision>
-	      <origin xyz="0 0 0.025" rpy="0 0 0"/>
-	      <geometry>
-		<box size="0.05 0.05 0.05"/>
-	      </geometry>
-	    </collision>
-	    <visual>
-	      <origin xyz="0 0 0.025" rpy="0 0 0"/>
-	      <geometry>
-		<box size="0.05 0.05 0.05"/>
-	      </geometry>
-	      <material name="red">
-		<color rgba="1 0 0 1"/>
-	      </material>
-	    </visual>
-	    <inertial>
-	      <mass value="1e-5" />
-	      <origin xyz="0 0 0" rpy="0 0 0"/>
-	      <inertia ixx="1e-6" ixy="0" ixz="0" iyy="1e-6" iyz="0" izz="1e-6" />
-	    </inertial>
-  </link>
+  	<inertial>
+  		<mass value="0.001"/>
+  		<origin xyz="0 0 0" rpy="0 0 0" />
+  		<inertia ixx="0.00000416666667" ixy="0" ixz="0" iyy="0.00000416666667" iyz="0" izz="0.00000416666667"/>
+  	</inertial>
+  	<collision>
+  	  <origin xyz="0 0 0.025" rpy="0 0 0"/>
+      <geometry>
+        <box size="0.05 0.05 0.05"/>
+      </geometry>
+  	</collision>
+  	<visual>
+  	  <origin xyz="0 0 0.025" rpy="0 0 0"/>
+      <geometry>
+        <box size="0.05 0.05 0.05"/>
+      </geometry>
+      <material name="white" />
+  	</visual>
+  </link>
+  <joint name="neck_joint" type="revolute">
+  	<axis xyz="0 0 1"/>
+  	<limit effort="1000.0" lower="-6.28" upper="6.28" velocity="0.2"/>
+  	<origin rpy="0 0 0" xyz="0 0 0.05"/>
+  	<parent link="neck_base_link"/>
+  	<child link="neck_link"/>
+  </joint>
   <joint name="camera_joint" type="fixed">
-	    <axis xyz="0 1 0" />
-	    <origin xyz="0.23 0 0.0" rpy="0 0 0"/>
-	    <parent link="link_chassis"/>
-	    <child link="camera_link"/>
-	 </joint>
+  	<origin rpy="0 0 0" xyz="0.0 0 0.25"/>
+  	<parent link="neck_link"/>
+  	<child link="camera_link"/>
+  </joint>
+<transmission name="neck_joint_trans">
+	<type>transmission_interface/SimpleTransmission</type>
+	<joint name="neck_joint">
+		<hardwareInterface>hardware_interface/EffortJointInterface</hardwareInterface>
+	</joint>
+	<actuator name="motor1">
+		<hardwareInterface>hardware_interface/EffortJointInterface</hardwareInterface>
+		<mechanicalInterface>1</mechanicalInterface>
+	</actuator>
+</transmission>
 </robot>

Commit message: robot to follow basic concept

File: urdf/robot.xacro (robot description, xacro)
@@ -125,4 +125,7 @@
     </visual>
   </link>
+  <!--###############################################
+                Joint definitions
+  ####################################################-->
   <joint name="joint_back_right_wheel" type="continuous">
     <origin rpy="0 0 0" xyz="-0.20 0.15 0"/>
@@ -203,4 +206,11 @@
   	</visual>
   </link>
+  <joint name="neck_joint" type="revolute">
+  	<axis xyz="0 0 1"/>
+  	<limit effort="1000.0" lower="-6.28" upper="6.28" velocity="0.2"/>
+  	<origin rpy="0 0 0" xyz="0 0 0.05"/>
+  	<parent link="neck_base_link"/>
+  	<child link="neck_link"/>
+  </joint>
   <link name="camera_link">
   	<inertial>
@@ -210,26 +220,19 @@
   	</inertial>
   	<collision>
-  	  <origin xyz="0 0 0.025" rpy="0 0 0"/>
-      <geometry>
-        <box size="0.05 0.05 0.05"/>
+  	  <origin xyz="0.05 0 0.025" rpy="0 0 0"/>
+      <geometry>
+        <box size="0.15 0.05 0.05"/>
       </geometry>
   	</collision>
   	<visual>
-  	  <origin xyz="0 0 0.025" rpy="0 0 0"/>
-      <geometry>
-        <box size="0.05 0.05 0.05"/>
+  	  <origin xyz="0.05 0 0.025" rpy="0 0 0"/>
+      <geometry>
+        <box size="0.15 0.05 0.05"/>
       </geometry>
       <material name="white" />
   	</visual>
   </link>
-  <joint name="neck_joint" type="revolute">
-  	<axis xyz="0 0 1"/>
-  	<limit effort="1000.0" lower="-6.28" upper="6.28" velocity="0.2"/>
-  	<origin rpy="0 0 0" xyz="0 0 0.05"/>
-  	<parent link="neck_base_link"/>
-  	<child link="neck_link"/>
-  </joint>
   <joint name="camera_joint" type="fixed">
-  	<origin rpy="0 0 0" xyz="0.0 0 0.25"/>
+  	<origin rpy="0 0 0" xyz="0 0 0.25"/>
   	<parent link="neck_link"/>
   	<child link="camera_link"/>

Commit message: camera control

File: urdf/robot.xacro (robot description, xacro)
@@ -63,5 +63,5 @@
       <material name="blue"/>
     </visual>
-    <!-- caster front
+    <!-- caster front -->
     <collision name="caster_front_collision">
       <origin rpy=" 0 0 0" xyz="0.35 0 -0.05"/>
@@ -75,5 +75,19 @@
         <sphere radius="0.05"/>
       </geometry>
-    </visual>-->
+    </visual>
+    <!---->
+    <!-- caster back for support -->
+    <collision name="caster_back_collision">
+      <origin rpy=" 0 0 0" xyz="-0.35 0 -0.05"/>
+      <geometry>
+        <sphere radius="0.05"/>
+      </geometry>
+    </collision>
+    <visual name="caster_back_visual">
+      <origin rpy=" 0 0 0" xyz="-0.2 0 -0.05"/>
+      <geometry>
+        <sphere radius="0.05"/>
+      </geometry>
+    </visual>
   </link>
   <link name="link_back_right_wheel">
@@ -101,4 +115,5 @@
     </visual>
   </link>
+ <!--
    <link name="link_front_right_wheel">
     <xacro:default_inertial mass="0.2"/>
@@ -125,9 +140,10 @@
     </visual>
   </link>
+-->
   <!--###############################################
                 Joint definitions
   ####################################################-->
   <joint name="joint_back_right_wheel" type="continuous">
-    <origin rpy="0 0 0" xyz="-0.20 0.15 0"/>
+    <origin rpy="0 0 0" xyz="-0.0 0.15 0"/>
     <child link="link_back_right_wheel"/>
     <parent link="link_chassis"/>
@@ -137,5 +153,5 @@
   </joint>
   <joint name="joint_back_left_wheel" type="continuous">
-    <origin rpy="0 0 0" xyz="-0.20 -0.15 0"/>
+    <origin rpy="0 0 0" xyz="-0.0 -0.15 0"/>
     <child link="link_back_left_wheel"/>
     <parent link="link_chassis"/>
@@ -144,4 +160,5 @@
     <joint_properties damping="1.0" friction="1.0"/>
   </joint>
+<!--
   <joint name="joint_front_right_wheel" type="continuous">
     <origin rpy="0 0 0" xyz="0.20 0.15 0"/>
@@ -160,4 +177,5 @@
     <joint_properties damping="1.0" friction="1.0"/>
   </joint>
+-->
 <!--camera links - neck definition -->
   <link name="neck_base_link">

Commit message: robot model update

File: urdf/robot.xacro (robot description, xacro)
@@ -77,5 +77,5 @@
     </visual>
     <!---->
-    <!-- caster back for support -->
+    <!-- caster back for support
     <collision name="caster_back_collision">
       <origin rpy=" 0 0 0" xyz="-0.35 0 -0.05"/>
@@ -85,9 +85,9 @@
     </collision>
     <visual name="caster_back_visual">
-      <origin rpy=" 0 0 0" xyz="-0.2 0 -0.05"/>
-      <geometry>
-        <sphere radius="0.05"/>
-      </geometry>
-    </visual>
+      <origin rpy=" 0 0 0" xyz="-0.35 0 -0.05"/>
+      <geometry>
+        <sphere radius="0.05"/>
+      </geometry>
+    </visual>-->
   </link>
   <link name="link_back_right_wheel">
@@ -145,5 +145,5 @@
   ####################################################-->
   <joint name="joint_back_right_wheel" type="continuous">
-    <origin rpy="0 0 0" xyz="-0.0 0.15 0"/>
+    <origin rpy="0 0 0" xyz="-0.05 0.15 0"/>
     <child link="link_back_right_wheel"/>
     <parent link="link_chassis"/>
@@ -153,5 +153,5 @@
   </joint>
   <joint name="joint_back_left_wheel" type="continuous">
-    <origin rpy="0 0 0" xyz="-0.0 -0.15 0"/>
+    <origin rpy="0 0 0" xyz="-0.05 -0.15 0"/>
     <child link="link_back_left_wheel"/>
     <parent link="link_chassis"/>
@@ -181,5 +181,5 @@
   <link name="neck_base_link">
   	<inertial>
-  		<mass value="0.01"/>
+  		<mass value="0.001"/>
   		<origin xyz="0 0 0" rpy="0 0 0" />
   		<inertia ixx="0.0000416666667" ixy="0" ixz="0" iyy="0.0000416666667" iyz="0" izz="0.0000416666667"/>
@@ -200,5 +200,5 @@
   </link>
   <joint name="neck_base_to_chassis" type="fixed">
-  	<origin rpy="0 0 0" xyz="0 0 0.085"/>
+  	<origin rpy="0 0 0" xyz="0.10 0 0.085"/>
   	<parent link="link_chassis"/>
   	<child link="neck_base_link"/>
